File: pcb/Power.sch (KiCad schematic (older format))
At the start: 51 parts

Commit message: Copper is likely complete
Parts:
- removed C? (x2): 100u, symbol CPOL
- removed C? (x4): 10n, symbol C-0402
- removed D? (x2): SS12, symbol SS12
- removed DZ? (x2): BZX84B5V6, symbol BZX84C
- removed J?: PWRIN, symbol HEAD-M3
- removed J?: PWREN, symbol HEAD-M1
- removed JP?: MANUAL, symbol JUMPER
- removed L? (x2): 1m, symbol LFERR
- removed Q? (x2): PMV160UP, symbol PMV160UP
- removed Q?: MMUN2231L, symbol MMUN2231L
- removed Q? (x2): 2N7002, symbol 2N7002
- removed Q? (x2): MMBT3906, symbol MMBT3906
- removed Q?: 2N4403, symbol 2N4403
- removed Q?: MMBT3904, symbol MMBT3904
- removed Q?: 2N4401, symbol 2N4401
- removed R? (x4): 10k, symbol R-0402
- removed R? (x2): THERM, symbol THERM
- removed R? (x4): 1k, symbol R-0402
- removed R? (x2): 360, symbol R-0402
- added J5: PWR5V, conn:CONN_5-SIL, symbol HEAD-M5
- added Q4, Q5: PMV160UP, IPC-semi-nominal:SOT-23, symbol PMV160UP
- added Q6, Q7: 2N7002, IPC-semi-nominal:SOT-23, symbol 2N7002
- C10, C11, C12, C13: renamed from C?; footprint (none) -> IPC7351-Nominal:CAPC1005X55
- C14, C15, C16, C17: renamed from C?; footprint (none) -> passive:C-ALUM-5mm
- C6, C7, C8, C9: renamed from C?; footprint (none) -> IPC7351-Nominal:CAPC2012X70
- U2: renamed from U?; footprint (none) -> IPC7351-Nominal:SOIC127P600X175-9
- U3: renamed from U?; footprint (none) -> IPC7351-Nominal:SOP65P490X110-9A
Connections:
- net +10: now also Q4.2
- net +5: now also Q5.2
- net -10: now also Q7.2
- net -5: now also Q6.2
- net GND: now also U2.9 (PAD), J5.3, Q4.1, Q5.1, Q6.1, Q7.1
- new net: J5.1, Q4.3
- new net: J5.2, Q5.3
- new net: J5.4, Q6.3
- new net: J5.5, Q7.3
Other:
- note added: "To use basic linear regulator, jumper pins 1-2 and 4-5.\nTo power externally, supply +5V to pin 1 and -5V to pin 5."
