File: pcb/wcp52-output.sch (KiCad schematic (older format))
At the start: 28 parts

Commit message: Copper is likely complete
Parts:
- C1, C2: renamed from C?; footprint (none) -> IPC7351-Nominal:CAPC1005X55
- J1: renamed from J?; footprint (none) -> conn:CONN-2_CONSMA001
- J2: renamed from J?; footprint (none) -> conn:CONN_2-SIL
- J3: renamed from J?; value COAX -> OUT; footprint (none) -> conn:CONN-2_CONSMA001
- Q1, Q2, Q3: renamed from Q?; footprint (none) -> IPC-semi-nominal:SOT-23
- R1, R10, R11, R2, R3, R4, R5, R6, R7, R8, R9: renamed from R?; footprint (none) -> IPC7351-Nominal:RESC1005X40
- R12, R13, R14, R15, R16, R17: renamed from R?; footprint (none) -> IPC7351-Nominal:RESC1608X50
- U1: renamed from U?; footprint (none) -> IPC-semi-nominal:SOT-23-5
- U2: renamed from U?; footprint (none) -> IPC7351-Nominal:SOIC127P600X175-9
- U3: renamed from U?; footprint (none) -> IPC7351-Nominal:SOP65P490X110-9A
