File: pcb/wcp52-output.kicad_pcb (KiCad board)
At the start: 4 copper layers, 33 x 33 mm, 50 parts, among them J1 IN, J2 CTRL, J3 OUT, J5 PWR5V, Q1 MMBT3906, Q2 2N7002, Q3 2N7002, Q4 PMV160UP, Q5 PMV160UP, Q6 2N7002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

Commit message: Silkscreen touchups
Other:
- board text added: "+10"
- board text added: "+5"
- board text added: "-10"
- board text added: "-15dB"
- board text added: "-5"
- board text added: "200"
- board text added: "31dB"
- board text added: "GND"
- board text added: "MHz"
- board text added: "SPEED LIMIT"
