File: pcb/wcp52-output.kicad_pcb (KiCad board)
At the start: 4 copper layers, 33 x 33 mm, 50 parts, among them J1 IN, J2 CTRL, J3 OUT, J5 PWR5V, Q1 MMBT3906, Q2 2N7002, Q3 2N7002, Q4 PMV160UP, Q5 PMV160UP, Q6 2N7002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

Commit message: More PCB touchups
Other:
- board text added: "25dB"
- board text added: "NOV 2014"
- board text added: "OUTPUT AMP"
- board text added: "WCP52"
- board text removed: "31dB"
